File: Schematics/LineFollower/power.kicad_sch (KiCad schematic)
At the start: 15 parts, among them U2 AMS1117-3.3, U3 TPS563201

Commit message: Uploaded V1.0 of PCB
Parts:
- removed C6: 10u, symbol Device:C_Polarized_Small
- added C6: 22u, Capacitor_SMD:C_0805_2012Metric_Pad1.18x1.45mm_HandSolder, symbol Device:C
- added D3: vBatt, LED_SMD:LED_1206_3216Metric_Pad1.42x1.75mm_HandSolder, symbol Device:LED
- added R12: 4k7, Resistor_SMD:R_0805_2012Metric_Pad1.20x1.40mm_HandSolder, symbol Device:R
- C5: value 10u -> 100u; footprint (none) -> Capacitor_SMD:CP_Elec_6.3x5.4
- C7: renamed from C4; footprint (none) -> Capacitor_SMD:C_0805_2012Metric_Pad1.18x1.45mm_HandSolder
- C8: renamed from C2; footprint (none) -> Capacitor_SMD:C_0805_2012Metric_Pad1.18x1.45mm_HandSolder
- C9: renamed from C3; footprint (none) -> Capacitor_SMD:C_0805_2012Metric_Pad1.18x1.45mm_HandSolder
- L1: footprint (none) -> Inductor_SMD:L_Chilisin_BMRF00101040; Campo4 (none) -> BCIHP1040SC-3R3M
- R10: renamed from R3; footprint (none) -> Resistor_SMD:R_0805_2012Metric_Pad1.20x1.40mm_HandSolder
- R11: renamed from R2; footprint (none) -> Resistor_SMD:R_0805_2012Metric_Pad1.20x1.40mm_HandSolder
- R7: renamed from R5; footprint (none) -> Resistor_SMD:R_1206_3216Metric_Pad1.30x1.75mm_HandSolder
- R8: renamed from R6; footprint (none) -> Resistor_SMD:R_1206_3216Metric_Pad1.30x1.75mm_HandSolder
- R9: renamed from R4; value R -> 10k; footprint (none) -> Resistor_SMD:R_0805_2012Metric_Pad1.20x1.40mm_HandSolder
- U4: renamed from U5; footprint (none) -> modulos:5v-Reg
- renumbered U3 to U5
Connections:
- net GND: now also C6.2, D3.1 (K)
- net V_BATT: now also C6.1, R12.1
- new net: D3.2 (A), R12.2
