File: Schematics/LineFollower/LineFollower.kicad_sch (KiCad schematic)
At the start: 6 parts, among them J1 Conn_01x10_MountingPin, J1 VBATT_IN, U1 ESP32-WROOM-E

Commit message: Uploaded V1.0 of PCB
Parts:
- removed J1: VBATT_IN, symbol Connector_Generic:Conn_01x02
- removed U2: ~, symbol radiocontrol:4in1_esc_15A
- added C3, C4 (x2): 100nF, Capacitor_SMD:C_0805_2012Metric_Pad1.18x1.45mm_HandSolder, symbol Device:C_Small
- added D1, D2: WS2812B, LED_SMD:LED_WS2812B_PLCC4_5.0x5.0mm_P3.2mm, symbol LED:WS2812B
- added D4: 3v3, LED_SMD:LED_1206_3216Metric_Pad1.42x1.75mm_HandSolder, symbol Device:LED
- added J2: StartModule, Connector_PinHeader_2.54mm:PinHeader_1x04_P2.54mm_Vertical, symbol Connector_Generic:Conn_01x04
- added J3: 4en1, Connector_JST:JST_SH_SM06B-SRSS-TB_1x06-1MP_P1.00mm_Horizontal, symbol Connector_Generic_MountingPin:Conn_01x06_MountingPin
- added J4: UART, Connector_PinHeader_2.54mm:PinHeader_1x04_P2.54mm_Vertical, symbol Connector_Generic:Conn_01x04
- added JP1: BOOT_SELECT, Connector_PinHeader_2.54mm:PinHeader_1x03_P2.54mm_Vertical, symbol Jumper:Jumper_3_Bridged12
- added R1: 4k7, Resistor_SMD:R_0805_2012Metric_Pad1.20x1.40mm_HandSolder, symbol Device:R
- added R12: 470, Resistor_SMD:R_0805_2012Metric_Pad1.20x1.40mm_HandSolder, symbol Device:R
- added R13, R4: 1k, Resistor_SMD:R_0805_2012Metric_Pad1.20x1.40mm_HandSolder, symbol Device:R
- added R2, R3: 2k2, Resistor_SMD:R_0805_2012Metric_Pad1.20x1.40mm_HandSolder, symbol Device:R
- added SW1: SW_DIP_x04, Button_Switch_THT:SW_DIP_SPSTx04_Slide_9.78x12.34mm_W7.62mm_P2.54mm, symbol Switch:SW_DIP_x04
- added SW2: SW_Push, switches:SKPMANE010 _Silicone_6x6mm, symbol Switch:SW_Push
- added SW3: Push2, switches:SKPMANE010 _Silicone_6x6mm, symbol Switch:SW_Push
- added SW4: SW_Push_SPDT, switches:SS12D07VG2, symbol Switch:SW_Push_SPDT
- added SW5: Start, switches:SKPMANE010 _Silicone_6x6mm, symbol Switch:SW_Push
- C3: footprint Capacitor_SMD:C_1206_3216Metric_Pad1.33x1.80mm_HandSolder -> Capacitor_SMD:C_0805_2012Metric_Pad1.18x1.45mm_HandSolder
- J1: value Conn_01x10_MountingPin -> Morro
Connections:
- net +3V3: now also J2.1 (Pin_1), J4.1 (Pin_1), JP1.1 (A), R1.2, R13.1, R2.2, R4.2, SW1.5, SW4.1 (A)
- net +5V: now also C3.1, C4.1, D1.1 (VDD), D2.1 (VDD)
- net GND: now also C3.2, C4.2, C4.2, D1.3 (VSS), D2.3 (VSS), D4.1 (K), J2.2 (Pin_2), J3.6 (Pin_6), J3.MP (MountPin), J4.4 (Pin_4), JP1.3 (B), R3.1, SW2.1, SW3.2, SW5.2
- net MOSFET_PWM: now also U1.12 (ADC2_CH7/GPIO27)
- net SCL: now also U1.10 (DAC_1/ADC2_CH8/GPIO25)
- net SDA: now also U1.11 (DAC_2/ADC2_CH9/GPIO26)
- net V1: now also U1.8 (32K_XP/GPIO32/ADC1_CH4)
- net V2: now also U1.9 (32K_XN/GPIO33/ADC1_CH5)
- net V_BATT_SENSE: now also U1.4 (SENSOR_VP/GPIO36/ADC1_CH0)
- net at C3.1, R12.1, U1.3 (EN/CHIP_PU): now also SW2.2
- net START: now reaches U1.13 (MTMS/GPIO14/ADC2_CH6)
- net START: now also J2.3 (Pin_3)
- net at U1.24 (ADC2_CH2/GPIO2): now also SW3.1
- net BOOT_SELECT: now reaches U1.25 (GPIO0/BOOT/ADC2_CH1)
- net BOOT_SELECT: now also JP1.2 (C)
- net MOTOR_1: now reaches U1.27 (GPIO16)
- net MOTOR_1: now also J3.1 (Pin_1)
- net MOTOR_2: now reaches U1.28 (GPIO17)
- net MOTOR_2: now also J3.2 (Pin_2)
- net at U1.29 (GPIO5): now also SW5.1
- net MOTOR_3: now reaches U1.30 (GPIO18)
- net MOTOR_3: now also J3.3 (Pin_3)
- net MOTOR_4: now reaches U1.31 (GPIO19)
- net MOTOR_4: now also J3.4 (Pin_4)
- net RGB_PIN: now reaches U1.33 (GPIO21)
- net RGB_PIN: now also R12.2
- net UART_RX: now reaches U1.34 (U0RXD/GPIO3)
- net UART_RX: now also J4.2 (Pin_2)
- net UART_TX: now reaches U1.35 (U0TXD/GPIO1)
- net UART_TX: now also J4.3 (Pin_3)
- net ENC_1A: now reaches U1.36 (GPIO22)
- net ENC_1B: now reaches U1.37 (GPIO23)
- net CONFIG: now reaches U1.5 (SENSOR_VN/GPIO39/ADC1_CH3)
- net CONFIG: now also C4.1, R3.2, SW1.1, SW1.2, SW1.3, SW1.4
- net ENC_2A: now reaches U1.6 (GPIO34/ADC1_CH6)
- net ENC_2B: now reaches U1.7 (GPIO35/ADC1_CH7)
- new net: R4.1, SW1.6
- new net: R2.1, SW1.7
- new net: R1.1, SW1.8
- new net: D1.2 (DOUT), D2.4 (DIN)
- new net: D4.2 (A), R13.2
- new net: D1.4 (DIN), R12.1
- new net KILL: J2.4 (Pin_4)
- new net Power/3v3: SW4.2 (B)
- new net V_BATT: J3.5 (Pin_5)
- no-connect marks 2 -> 8
Other:
- moved on the sheet: C3, J1, R12, U1

Commit message: Version 1.1 PCB: Fixed I2C pullups
Parts:
- added R14, R15: 2k, Resistor_SMD:R_1206_3216Metric_Pad1.30x1.75mm_HandSolder, symbol Device:R
Connections:
- net +3V3: now also R14.2, R15.2
- net SCL: now also R14.1
- net SDA: now also R15.1
